Commit message: modified launch files

File: Day6/catkin_ws/src/my_first_robot/urdf/my_robot.xacro (robot description, xacro)
@@ -2,4 +2,9 @@
 <robot name="my_first_robot" xmlns:xacro="http://www.ros.org/wiki/xacro">
     <xacro:include filename="$(find my_first_robot)/urdf/my_robot.gazebo"/>
+    <link name="base_link" />
+    <joint name="base_link_to_chassis" type="fixed">
+    <parent link="base_link"/>
+    <child link="chassis"/>
+    </joint>
     <link name="chassis">
         <inertial>
@@ -49,5 +54,5 @@
     </link>
     <joint name="chassis_to_right_wheel" type="continuous">
-        <origin rpy="0 0.0 0.0" xyz="0.0 0.275 -0.03"/>
+        <origin rpy="0 0.0 0.0" xyz="0.0 -0.275 -0.03"/>
         <parent link="chassis"/>
         <child link="right_wheel"/>
@@ -79,5 +84,5 @@
     </link>
     <joint name="chassis_to_left_wheel" type="continuous">
-        <origin rpy="0 0.0 0.0" xyz="0.0 -0.275 -0.03"/>
+        <origin rpy="0 0.0 0.0" xyz="0.0 0.275 -0.03"/>
         <parent link="chassis"/>
         <child link="left_wheel"/>
